File: HARDWARE/LiPower-Shield.brd (EAGLE design)
At the start: 59.7 x 53.3 mm, 52 parts, among them U1 MAX17043G+U, U2 TPS61200, U3 MCP73831, U4 ARDUINO_R3_SHIELD, X1 USBSMD

Commit message: Schematic Cleanup
fixed all of these...

1) GND and 5V symbols need to be rotated "up" and "down".

2) all LEDs prefixes should be "D#"

3) R4 needs to be shifted down one grid space. The resulting 4 way
junction will need to be fixed then too.

4) J1 should have a prefix of JP#

5) USB connector is currently "X1" should be a JP prefix.

6) small flame symbol needs to be updated.
Parts:
- removed JP100: LOGO-SFESK, SparkFun:SFE-LOGO-FLAME
- added LOGO3: SFE_LOGO_FLAME.1_INCH, SparkFun-Aesthetics:SFE_LOGO_FLAME_.1
- renumbered J1 to JP, LED1 to D1, LED2 to D2, X1 to JP11
Routing:
- net 5V: track 69.6 -> 67.8 mm
Changed lines of the file:
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@@
 <layer number="29" name="tStop" color="7" fill="3" visible="no" active="yes"/>
 <layer number="30" name="bStop" color="7" fill="6" visible="no" active="yes"/>
-<layer number="31" name="tCream" color="7" fill="4" visible="yes" active="yes"/>
+<layer number="31" name="tCream" color="7" fill="4" visible="no" active="yes"/>
 <layer number="32" name="bCream" color="7" fill="5" visible="no" active="yes"/>
 <layer number="33" name="tFinish" color="6" fill="3" visible="no" active="yes"/>
@@
 <attribute name="PROD_ID" value="IC-09995" x="13.97" y="38.1" size="1.778" layer="27" rot="R90" display="off"/>
 </element>
-<element name="X1" library="SparkFun-Connectors" package="USB-MINIB" value="USBSMD" x="5.08" y="38.1">
+<element name="JP11" library="SparkFun-Connectors" package="USB-MINIB" value="USBSMD" x="5.08" y="38.1">
 <attribute name="PROD_ID" value="CONN-08193" x="5.08" y="38.1" size="1.778" layer="27" display="off"/>
 </element>
@@
 <attribute name="VALUE" value="330" x="20.32" y="33.782" size="1.778" layer="27" rot="R180" display="off"/>
 </element>
-<element name="LED2" library="SparkFun-LED" package="LED-0603" value="RED" x="20.2946" y="35.3314" rot="R270">
+<element name="D2" library="SparkFun-LED" package="LED-0603" value="RED" x="20.2946" y="35.3314" rot="R270">
 <attribute name="PROD_ID" value="DIO-00819" x="20.2946" y="35.3314" size="1.778" layer="27" rot="R270" display="off"/>
 <attribute name="VALUE" value="RED" x="20.2946" y="35.3314" size="1.778" layer="27" rot="R270" display="off"/>
@@
 <element name="JP1" library="SparkFun" package="1X02_NO_SILK" value="" x="1.27" y="8.89" rot="R90"/>
 <element name="SJ1" library="SparkFun" package="SJ_2S-TRACE" value="SOLDERJUMPERTRACE" x="19.05" y="30.48" rot="MR90"/>
-<element name="JP100" library="SparkFun" package="SFE-LOGO-FLAME" value="LOGO-SFESK" x="55.69458125" y="10.855959375"/>
 <element name="R2" library="SparkFun-Resistors" package="0603-RES" value="4.7k" x="19.05" y="6.35" rot="R90">
 <attribute name="PROD_ID" value="RES-07857" x="19.05" y="6.35" size="1.778" layer="27" rot="R90" display="off"/>
@@
 <attribute name="VALUE" value="1.0uF" x="15.875" y="13.9954" size="1.778" layer="27" rot="R90" display="off"/>
 </element>
-<element name="LED1" library="SparkFun-LED" package="LED-0603" value="RED" x="19.05" y="16.51" rot="R270">
+<element name="D1" library="SparkFun-LED" package="LED-0603" value="RED" x="19.05" y="16.51" rot="R270">
 <attribute name="PROD_ID" value="DIO-00819" x="19.05" y="16.51" size="1.778" layer="27" rot="R270" display="off"/>
 <attribute name="VALUE" value="RED" x="19.05" y="16.51" size="1.778" layer="27" rot="R270" display="off"/>
@@
 <element name="JP5" library="abes" package="FIDUCIAL-1X2.5" value="FIDUCIAL1X2.5" x="1.27" y="49.53"/>
 <element name="JP6" library="abes" package="FIDUCIAL-1X2.5" value="FIDUCIAL1X2.5" x="58.42" y="10.16"/>
-<element name="J1" library="SparkFun-Connectors" package="JST-2-SMD" value="" x="5.717540625" y="10.182859375" rot="R90">
+<element name="JP" library="SparkFun-Connectors" package="JST-2-SMD" value="" x="5.717540625" y="10.182859375" rot="R90">
 <attribute name="PROD_ID" value="CONN-08352" x="5.717540625" y="10.182859375" size="1.778" layer="27" rot="R90" display="off"/>
 </element>
@@
 <element name="JP9" library="SparkFun" package="STAND-OFF-TIGHT" value="STAND-OFFTIGHT" x="5.08" y="50.8"/>
 <element name="JP10" library="SparkFun" package="STAND-OFF-TIGHT" value="STAND-OFFTIGHT" x="57.15" y="6.35"/>
+<element name="LOGO3" library="SparkFun-Aesthetics" package="SFE_LOGO_FLAME_.1" value="SFE_LOGO_FLAME.1_INCH" x="55.372" y="10.541"/>
 </elements>
 <signals>
 <signal name="GND">
-<contactref element="X1" pad="GND"/>
+<contactref element="JP11" pad="GND"/>
 <contactref element="C8" pad="1"/>
 <contactref element="U3" pad="2"/>
@@
 <contactref element="C2" pad="2"/>
 <contactref element="JP4" pad="2"/>
-<contactref element="LED1" pad="C"/>
 <contactref element="C4" pad="2"/>
 <contactref element="U2" pad="15"/>
@@
 <vertex x="59.69" y="0"/>
 </polygon>
-<contactref element="J1" pad="1"/>
+<contactref element="JP" pad="1"/>
 <wire x1="9.095" y1="24.63" x2="8.12" y2="24.63" width="0.254" layer="1"/>
 <wire x1="8.12" y1="24.63" x2="7.62" y2="24.13" width="0.254" layer="1"/>
@@
 <via x="7.6327" y="23.70328125" extent="1-16" drill="0.381"/>
 <contactref element="R9" pad="1"/>
+<contactref element="D1" pad="C"/>
 </signal>
 <signal name="PROG">
@@
 <signal name="N$5">
 <contactref element="R12" pad="1"/>
-<contactref element="LED2" pad="C"/>
+<contactref element="D2" pad="C"/>
 <wire x1="21.1446" y1="35.3044" x2="21.1716" y2="35.3314" width="0.254" layer="1"/>
 <wire x1="21.1446" y1="35.3044" x2="21.1446" y2="33.8074" width="0.254" layer="1"/>
@@
 <signal name="5V">
 <contactref element="U4" pad="5V"/>
-<contactref element="R3" pad="1"/>
-<contactref element="U2" pad="2"/>
 <contactref element="R4" pad="2"/>
-<contactref element="C3" pad="1"/>
 <wire x1="21.614903125" y1="29.185096875" x2="19.05" y2="31.75" width="0.254" layer="1"/>
 <wire x1="21.59" y1="6.35" x2="22.86" y2="5.08" width="0.254" layer="1"/>
@@
 <wire x1="7.4676" y1="31.75" x2="6.35" y2="31.75" width="0.254" layer="1"/>
 <wire x1="7.4676" y1="31.75" x2="7.4676" y2="28.79" width="0.254" layer="1"/>
-<wire x1="6.145" y1="24.63" x2="5.0118" y2="24.63" width="0.254" layer="1"/>
 <wire x1="5.0118" y1="24.63" x2="4.318" y2="25.3238" width="0.254" layer="1"/>
 <wire x1="4.318" y1="25.3238" x2="4.318" y2="27.94" width="0.254" layer="1"/>
 <wire x1="4.318" y1="27.94" x2="4.318" y2="29.718" width="0.254" layer="1"/>
 <wire x1="4.318" y1="29.718" x2="6.35" y2="31.75" width="0.254" layer="1"/>
-<wire x1="3.1606" y1="27.94" x2="4.318" y2="27.94" width="0.254" layer="1"/>
-<wire x1="19.9" y1="18.034" x2="21.614903125" y2="18.034" width="0.254" layer="1"/>
 <wire x1="21.59" y1="6.35" x2="21.59" y2="10.9982" width="0.254" layer="1"/>
 <wire x1="21.59" y1="10.9982" x2="22.4028" y2="11.811" width="0.254" layer="1"/>
@@
 <wire x1="29.21" y1="5.08" x2="29.21" y2="2.54" width="0.254" layer="1"/>
 <wire x1="22.86" y1="5.08" x2="29.21" y2="5.08" width="0.254" layer="1"/>
+<contactref element="U2" pad="2"/>
+<contactref element="C3" pad="1"/>
+<wire x1="3.1606" y1="27.94" x2="4.318" y2="27.94" width="0.254" layer="1"/>
+<wire x1="5.0118" y1="24.63" x2="6.145" y2="24.63" width="0.254" layer="1"/>
+<contactref element="R3" pad="1"/>
+<wire x1="21.614903125" y1="18.008103125" x2="19.9" y2="18.034" width="0" layer="19" extent="1-1"/>
 </signal>
 <signal name="3.3V">
@@
 </signal>
 <signal name="VBUS">
-<contactref element="X1" pad="VBUS"/>
-<contactref element="LED2" pad="A"/>
+<contactref element="JP11" pad="VBUS"/>
+<contactref element="D2" pad="A"/>
 <contactref element="C8" pad="2"/>
 <contactref element="U3" pad="4"/>
@@
 </signal>
 <signal name="N$1">
-<contactref element="LED1" pad="A"/>
+<contactref element="D1" pad="A"/>
 <contactref element="R3" pad="2"/>
 <wire x1="18.173" y1="16.51" x2="18.2" y2="16.537" width="0.254" layer="1"/>
@@
 <signal name="N$7">
 <contactref element="JP1" pad="2"/>
-<contactref element="J1" pad="2"/>
+<contactref element="JP" pad="2"/>
 <contactref element="S2" pad="2"/>
 <wire x1="5.08" y1="11.16" x2="1.54" y2="11.16" width="0.508" layer="1"/>

Commit message: changed fids to regular from micro
Parts:
- removed JP5, JP6: FIDUCIAL1X2.5, abes:FIDUCIAL-1X2.5
- added FID1, FID2: FIDUCIAL1X2, SparkFun-Aesthetics:FIDUCIAL-1X2

Commit message: Fixed current QC checklist issues.
Parts:
- renumbered JP to JP13
Routing:
- net 5V: track 67.8 -> 69.6 mm
